Commit message: test

File: coco_one.urdf (robot description, URDF)
Before this commit: robot coco_one, 1 links, 0 joints
Links:
- link base_link: geometry visual mesh filename=https://raw.githubusercontent.com/MNowickixBerry/robot_mode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

Commit message: Scaling the model

File: coco_one.urdf (robot description, URDF)
Before this commit: robot coco_one, 1 links, 0 joints
Links:
- link base_link: geometry visual mesh filename=https://raw.githubusercontent.com/MNowickixBerry/robot_mode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 scale=0.001 0.001 0.001
